File: hardware/industrial-quad-relay.kicad_pcb (KiCad board)
At the start: 2 copper layers, 40 x 40 mm, 22 parts, among them P1 CON-SENSOR, P2 Digital_Output, U1 M24C64, U2 CPC1020N, U3 CPC1020N, U4 CPC1020N, U5 CPC1020N, U6 DRILL, U7 DRILL, U8 DRILL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

Commit message: Add 3d information (final)
Parts:
- C1: footprint 0603 -> kicad-libraries:C0603
- Fiducial_Mark (x2): footprint Fiducial_Mark -> kicad-libraries:Fiducial_Mark
- G***: footprint Logo_31x31 -> kicad-libraries:Logo_31x31
- P1: footprint CON-SENSOR -> kicad-libraries:CON-SENSOR
- P2: value Digital_Output -> Digital Output; footprint OQ_8P -> kicad-libraries:OQ_8P
- R1, R2, R3, R4: footprint 1210 -> kicad-libraries:R1210
- RP1: footprint 0603X4 -> kicad-libraries:0603X4
- U1: footprint SOIC8 -> kicad-libraries:SOIC8
- U2, U3, U4, U5: footprint SOP4 -> kicad-libraries:SOP4-WIDE
- U6, U7, U8, U9: footprint DRILL_NP -> kicad-libraries:DRILL_NP
- VAL: footprint CE_5mm -> kicad-libraries:CE_5mm
- VAL: footprint WEEE_7mm -> kicad-libraries:WEEE_7mm
Connections:
- P1 pad 1: (no net) -> Net-(P1-Pad1)
- U1 pad 7: (no net) -> Net-(U1-Pad7)
